Commit message: added pool

File: src/robot_description/model/robot.xacro (robot description, xacro)
@@ -20,6 +20,6 @@
                 <mesh filename="file://$(find robot_description)/meshes/base_link.stl" scale="0.001 0.001 0.001" />
             </geometry>
-            <material name="base_link_material">
-                <color rgba="0.5 0.5 0.5 1.0"/>
+            <material name="yellow_material">
+                <color rgba="1.0 1.0 0.0 1.0"/>
             </material>
         </visual>
@@ -42,6 +42,6 @@
                 <mesh filename="file://$(find robot_description)/meshes/canister_m1.stl" scale="0.001 0.001 0.001" />
             </geometry>
-            <material name="base_link_material">
-                <color rgba="0.5 0.5 0.5 1.0"/>
+            <material name="black_material">
+                <color rgba="0.0 0.0 0.0 1.0"/>
             </material>
         </visual>
@@ -64,6 +64,6 @@
                 <mesh filename="file://$(find robot_description)/meshes/canister_m2.stl" scale="0.001 0.001 0.001" />
             </geometry>
-            <material name="base_link_material">
-                <color rgba="0.5 0.5 0.5 1.0"/>
+            <material name="black_material">
+                <color rgba="0.0 0.0 0.0 1.0"/>
             </material>
         </visual>
@@ -86,4 +86,7 @@
                 <mesh filename="file://$(find robot_description)/meshes/cannister_s1.stl" scale="0.001 0.001 0.001" />
             </geometry>
+            <material name="black_material">
+                <color rgba="0.0 0.0 0.0 1.0"/>
+            </material>
         </visual>
         <collision name="cannister_s1_collision">
@@ -105,4 +108,7 @@
                 <mesh filename="file://$(find robot_description)/meshes/cannister_s2.stl" scale="0.001 0.001 0.001" />
             </geometry>
+            <material name="black_material">
+                <color rgba="0.0 0.0 0.0 1.0"/>
+            </material>
         </visual>
         <collision name="cannister_s2_collision">

Commit message: added camera

File: src/robot_description/model/robot.xacro (robot description, xacro)
@@ -215,4 +215,21 @@
         </collision>
     </link>
+    <link name ="camera_link">
+        <visual name="camera_visual">
+            <origin xyz="0.0 0.0 0.0" rpy="0.0 0.0 0.0" />
+            <geometry>
+                <box size="0.01 0.01 0.01" />
+            </geometry>
+            <material name="black_material">
+                <color rgba="0.0 0.0 0.0 1.0"/>
+            </material>
+        </visual>
+        <collision name="camera_collision">
+            <origin xyz="0.0 0.0 0.0" rpy="0.0 0.0 0.0" />
+            <geometry>
+                <box size="0.01 0.01 0.01" />
+            </geometry>
+        </collision>
+    </link>
     <joint name="base_link_Rigid-1" type="fixed">
         <origin xyz="0.125 0.0 0.07" rpy="0.0 -0.0 0.0" />
@@ -264,3 +281,8 @@
         <child link="stone" />
     </joint>
+    <joint name="base_link_Rigid-10" type="fixed">
+        <origin xyz="0.21 0.0 0.0" rpy="0.0 0.0 0.0" />
+        <parent link="base_link" />
+        <child link="camera_link" />
+    </joint>
 </robot>

Commit message: down camera

File: src/robot_description/model/robot.xacro (robot description, xacro)
@@ -232,4 +232,21 @@
         </collision>
     </link>
+    <link name ="camera_link_down">
+        <visual name="camera_down_visual">
+            <origin xyz="0.0 0.0 0.0" rpy="0.0 0.0 0.0" />
+            <geometry>
+                <box size="0.01 0.01 0.01" />
+            </geometry>
+            <material name="black_material">
+                <color rgba="0.0 0.0 0.0 1.0"/>
+            </material>
+        </visual>
+        <collision name="camera_down_collision">
+            <origin xyz="0.0 0.0 0.0" rpy="0.0 0.0 0.0" />
+            <geometry>
+                <box size="0.01 0.01 0.01" />
+            </geometry>
+        </collision>
+    </link>
     <joint name="base_link_Rigid-1" type="fixed">
         <origin xyz="0.125 0.0 0.07" rpy="0.0 -0.0 0.0" />
@@ -286,3 +303,8 @@
         <child link="camera_link" />
     </joint>
+    <joint name="base_link_Rigid-11" type="fixed">
+        <origin xyz="0.21 0.0 0.0" rpy="0.0 1.57 0.0" />
+        <parent link="base_link" />
+        <child link="camera_link_down" />
+    </joint>
 </robot>
